File: HP_2116_Logic_Regulator/HP_2116_Logic_Regulator.kicad_sch (KiCad schematic)
At the start: 122 parts, among them Q1 2N3906, Q2 2N3906, Q3 2N3906, Q30 2N1132, Q31 2N1132, Q32 2N1132, Q33 2N1305, Q34 2N1305, Q35 2N1132, Q36 2N1132, Q37 2N1305, Q38 2N1305, Q39 2N1711, Q4 2N3906, Q40 2N1711, Q41 AF Si Power, Q42 2N1304, Q43 2N1305, Q44 2N1304, Q5 2N3906, Q6 2N3906, Q7 2N3906, Q8 2N3904, Q9 2N3904

Commit message: Updated some values in the logic regulator and re-generated the svg and created pdfs.
Parts:
- removed D3, D4: D_Small, symbol Device:D_Small
- removed R11: 1k, symbol Device:R_Small
- added D6: 1N4148, symbol Device:D_Small
- D1, D2, D5: value D_Small -> 1N4148
- R1, R12, R3, R6, R7: value 1k -> 4.7k
- R10, R14: value 1k -> 470
- R13, R2, R4, R5, R8, R9: value 10k -> 2.2k
- R15, R16: value 470 -> 220
- R17: value 2.2k -> 470
Connections:
- net at Q5.2 (B), R9.1: now also Q7.2 (B), D6.2 (A); no longer D1.2 (A)
- new net: D1.2 (A), D6.1 (K)
Other:
- moved on the sheet: D1, D2

Commit message: Started to do a layout.
Parts:
- removed Q30, Q31, Q32, Q35, Q36: 2N1132, symbol Simulation_SPICE:PNP
- removed Q33, Q34, Q38, Q43: 2N1305, symbol Simulation_SPICE:PNP
- removed Q39, Q40: 2N1711, symbol Simulation_SPICE:NPN
- removed Q41: AF Si Power, symbol Simulation_SPICE:NPN
- removed Q42: 2N1304, symbol Simulation_SPICE:NPN
- added C45, C47, C48, C49: 100n, Capacitor_THT:C_Disc_D4.3mm_W1.9mm_P5.00mm, symbol Device:C_Small
- added C58: 1n, Capacitor_THT:C_Disc_D4.3mm_W1.9mm_P5.00mm, symbol Device:C_Small
- added H1: MountingHole, MountingHole:MountingHole_3.7mm, symbol Mechanical:MountingHole
- added Q30, Q31, Q32, Q35, Q36: 2N1132, Package_TO_SOT_THT:TO-5-3, symbol Transistor_BJT:Q_PNP_EBC
- added Q33, Q34, Q38, Q43: 2N1305, Package_TO_SOT_THT:TO-5-3, symbol Transistor_BJT:Q_PNP_EBC
- added Q39, Q40: 2N1711, Package_TO_SOT_THT:TO-5-3, symbol Transistor_BJT:Q_NPN_EBC
- added Q41: TIP41, Package_TO_SOT_THT:TO-220-3_Horizontal_TabDown, symbol Transistor_BJT:Q_NPN_BCE
- added Q42: 2N1304, Package_TO_SOT_THT:TO-5-3, symbol Transistor_BJT:Q_NPN_EBC
- C40, C41, C42, C43, C44, C46, C50, C51, C52: footprint (none) -> Capacitor_THT:C_Disc_D4.3mm_W1.9mm_P5.00mm
- C53, C55, C57: footprint (none) -> Capacitor_THT:CP_Radial_D5.0mm_P2.00mm
- C54: footprint (none) -> Capacitor_THT:CP_Radial_D16.0mm_P7.50mm
- C56: footprint (none) -> Capacitor_THT:CP_Radial_D6.3mm_P2.50mm
- CR50, CR52: footprint (none) -> Diode_THT:D_DO-41_SOD81_P10.16mm_Horizontal
- CR51, CR53, CR54, CR55, CR56, CR57, CR58, CR60, CR61, CR62, CR63, CR64, CR65, D1, D2, D6: footprint (none) -> Diode_THT:D_DO-35_SOD27_P10.16mm_Horizontal
- CR59: renamed from D5; footprint (none) -> Diode_THT:D_DO-35_SOD27_P10.16mm_Horizontal
- J1: footprint (none) -> HP_Connector:22 Pin HP EDAC
- Q37, Q44: footprint (none) -> Package_TO_SOT_THT:TO-5-3
- R1, R10, R100, R102, R103, R110, R111, R112, R113, R114, R115, R116, R117, R118, R119, R12, R13, R14, R15, R16, R17, R2, R3, R4, R5, R6, R61, R63, R64, R65, R67, R68, R7, R70, R71, R72, R74, R75, R77, R78, R8, R81, R82, R83, R85, R86, R87, R89, R9, R98, R99: footprint (none) -> Resistor_THT:R_Axial_DIN0207_L6.3mm_D2.5mm_P10.16mm_Horizontal
- R101, R62, R88: footprint (none) -> Resistor_THT:R_Axial_DIN0414_L11.9mm_D4.5mm_P20.32mm_Horizontal
- R66, R69, R76, R84, R96: footprint (none) -> Potentiometer_THT:Potentiometer_Bourns_3266W_Vertical
- R80: renamed from R90; footprint (none) -> Resistor_THT:R_Axial_DIN0207_L6.3mm_D2.5mm_P10.16mm_Horizontal
- R95, R97: footprint (none) -> Resistor_THT:R_Axial_DIN0309_L9.0mm_D3.2mm_P15.24mm_Horizontal
Connections:
- net +12VREGDRV: now also Q41.3 (E)
- net +20V: now also Q40.3 (C)
- net +23.3V: now also Q41.2 (C)
- net +4.5V: now also Q30.2 (B)
- net +4.5VREGDRV: now also Q32.1 (E)
- net -12.4V: now also C47.2, Q32.3 (C)
- net -12V: now also Q42.1 (E)
- net -20V: now also C45.2
- net -2V_E5: now also C48.2
- net -2V_R: now also C49.2, Q38.1 (E)
- net GND: now also C45.1, C47.1, C48.1, C49.1, C58.1, Q34.2 (B), Q36.2 (B), Q39.1 (E), Q43.1 (E)
- net GND_14: now also Q33.1 (E)
- net at C52.2, R100.1, R99.2: now also Q39.3 (C), Q42.3 (C)
- net at R100.2: now also Q40.2 (B)
- net at R78.2, R80.2, R81.1: now also C58.2, Q35.3 (C), Q38.3 (C)
- net at C50.1, R76.2: now also Q35.2 (B)
- net at R74.1: now also Q35.1 (E), Q36.1 (E)
- net at R101.1: now also Q40.1 (E), Q41.1 (B)
- net at C46.1, R66.2: now also Q31.2 (B)
- net at R63.2: now also Q30.1 (E), Q31.1 (E)
- net at R111.2, R112.2: now also Q43.2 (B)
- net at C44.2, R64.1, R68.1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: now also Q31.3 (C), Q33.3 (C), Q34.3 (C)
- net at C53.1, R85.2, R86.2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: now also Q38.2 (B)
- net at C55.1, R102.2, R103.2: now also Q42.2 (B)
- net at R110.1: now also Q43.3 (C)
- net at R68.2: now also Q32.2 (B)
- net at R96.2, R98.2: now also Q39.2 (B)
- net at C57.1, R70.2, R71.2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: now also Q33.2 (B)
- net at CR54.2 (A), R83.1: now also Q34.1 (E)
- net at CR51.2 (A): now also Q30.3 (C)
- net at CR53.2 (A): now also Q36.3 (C)
