File: HP_2116_Memory_Regulator/HP_2116_Memory_Regulator.kicad_sch (KiCad schematic)
At the start: 80 parts, among them Q50 2N3906, Q51 2N3906, Q52 2N4037, Q53 2N1305, Q54 2N4044, Q55 S17843, Q56 2N1304, Q57 2N3906, Q58 2N3906, Q59 2N4037, Q60 2N1305, Q61 2N4044, Q62 S17843, Q63 2N3054, Q64 2N1304

Commit message: Started to do a layout.
Parts:
- added H1: MountingHole, MountingHole:MountingHole_3.7mm, symbol Mechanical:MountingHole
- C70, C71, C72, C73, C74, C75, C76, C77, C78, C79, C80, C81: footprint (none) -> Capacitor_THT:C_Disc_D4.3mm_W1.9mm_P5.00mm
- CR70, CR71, CR72, CR73, CR74: footprint (none) -> Diode_THT:D_DO-41_SOD81_P10.16mm_Horizontal
- J1: footprint (none) -> HP Connector:Untitled
- Q50, Q51, Q57, Q58: footprint (none) -> Package_TO_SOT_THT:TO-92_Inline; symbol Device:Q_PNP -> Transistor_BJT:Q_PNP_EBC
- Q52, Q53, Q60: footprint (none) -> Package_TO_SOT_THT:TO-5-3; symbol Device:Q_PNP -> Transistor_BJT:Q_PNP_EBC
- Q54, Q61: footprint (none) -> Package_TO_SOT_THT:TO-78-6
- Q55, Q62: footprint (none) -> Package_TO_SOT_THT:TO-5-3
- Q56, Q64: footprint (none) -> Package_TO_SOT_THT:TO-5-3; symbol Transistor_BJT:Q_NPN_BCE -> Transistor_BJT:Q_NPN_EBC
- Q59: footprint (none) -> Package_TO_SOT_THT:TO-5-3; symbol Device:Q_PNP -> Transistor_BJT:Q_NPN_EBC
- Q63: value 2N3054 -> 2N3054 (TIP41); footprint (none) -> Package_TO_SOT_THT:TO-220-3_Horizontal_TabDown
- R125, R140, R155, R170: footprint (none) -> Potentiometer_THT:Potentiometer_Bourns_3266W_Vertical
- R126, R127, R128, R129, R130, R131, R132, R133, R134, R135, R141, R142, R143, R144, R145, R146, R147, R148, R149, R156, R157, R158, R159, R160, R161, R162, R163, R164, R171, R172, R173, R174, R175, R176, R177, R178, R179, R180, R181: footprint (none) -> Resistor_THT:R_Axial_DIN0207_L6.3mm_D2.5mm_P10.16mm_Horizontal
- R136, R150, R165: footprint (none) -> Resistor_THT:R_Axial_DIN0414_L11.9mm_D4.5mm_P15.24mm_Horizontal
- R182: footprint (none) -> Resistor_THT:R_Axial_DIN0414_L11.9mm_D4.5mm_P25.40mm_Horizontal
Connections:
- net +22V: now also Q56.1 (E), Q64.1 (E); no longer Q56.3 (E), Q64.3 (E)
- net +40V: now also R144.1
- net -12V: now also Q51.3 (C), Q53.1 (E); no longer Q51.C, Q53.E
- net -12VDRIVE: now also Q52.1 (E); no longer Q52.E
- net -12VSHUTOFF: now also Q50.3 (C); no longer Q50.C
- net -22.6V: now also Q52.3 (C); no longer Q52.C
- net -22V: now also Q58.3 (C), Q60.1 (E); no longer Q58.C, Q60.E
- net -22VDRIVE: now also Q59.1 (E); no longer Q59.E
- net -36.4V: now also Q59.3 (C); no longer Q59.C
- net GND: now also Q58.2 (B); no longer Q58.B
- net at R159.2, R161.1: now also Q57.3 (C); no longer Q57.C
- net at C77.1, R161.2, R162.1: now also Q59.2 (B); no longer Q59.B
- net at R134.1, R135.2: now also Q53.2 (B); no longer Q53.B
- net at C71.1, R132.2, R133.1: now also Q52.2 (B); no longer Q52.B
- net at R133.2: now also Q53.3 (C); no longer Q53.C
- net at R156.2, R157.2, R158.1: now also Q57.2 (B); no longer Q57.B
- net at CR70.2 (A), R131.1: now also Q51.2 (B); no longer Q51.B
- net at R147.2: now also Q56.3 (C); no longer Q56.2 (C)
- net at R163.2, R164.1: now also Q60.2 (B); no longer Q60.B
- net at R162.2: now also Q60.3 (C); no longer Q60.C
- net at R126.2, R127.2, R128.1: now also Q50.2 (B); no longer Q50.B
- net at R148.1, R149.1: now also Q56.2 (B); no longer Q56.1 (B)
- net at R180.1, R181.1: now also Q64.2 (B); no longer Q64.1 (B)
- net at R179.2: now also Q64.3 (C); no longer Q64.2 (C)
- new net: Q57.1 (E), Q58.1 (E), R160.1
- new net: Q50.1 (E), Q51.1 (E), R130.1
